Commit message: caster

File: ros2/src/mobile_robot/urdf/robot.urdf (robot description, URDF)
Before this commit: robot simple_diff_robot, 3 links, 2 joints
Links:
- removed link left_wheel
- removed link right_wheel
- added link caster, mass 0.1; collision sphere radius=0.03; visual sphere radius=0.03
- added link front_left_wheel, mass 0.5; collision cylinder length=0.03 radius=0.05; visual cylinder length=0.03 radius=0.05
- added link front_right_wheel, mass 0.5; collision cylinder length=0.03 radius=0.05; visual cylinder length=0.03 radius=0.05
- link base_link: geometry collision box size=0.5 0.4 0.1; visual box size=0.5 0.4 0.1
Joints:
- removed joint left_wheel_joint
- removed joint right_wheel_joint
- added joint caster_joint: type fixed, parent base_link, child caster, origin xyz=-0.2 0 -0.03
- added joint front_left_wheel_joint: type continuous, parent base_link, child front_left_wheel, origin xyz=0.2 0.215 -0.02, axis 0 1 0
- added joint front_right_wheel_joint: type continuous, parent base_link, child front_right_wheel, origin xyz=0.2 -0.215 -0.02, axis 0 1 0

Commit message: Init commit

File: ros2/src/mobile_robot/urdf/robot.urdf (robot description, URDF)
Before this commit: robot four_wheel_front_drive, 4 links, 3 joints
Links:
- added link camera_link
- added link ray_link
Joints:
- added joint camera_joint: type fixed, parent base_link, child camera_link, origin xyz=0.2 0 0.1 rpy=0 0 0
- added joint ray_joint: type fixed, parent base_link, child ray_link, origin xyz=0.2 0 0.1 rpy=0 0 0

Commit message: Add box to world, new model tests.

File: ros2/src/mobile_robot/urdf/robot.urdf (robot description, URDF)
Before this commit: robot four_wheel_front_drive, 6 links, 5 joints
Links:
- removed link camera_link
- removed link ray_link
- added link depth_camera_link
Joints:
- removed joint camera_joint
- removed joint ray_joint
- added joint depth_camera_joint: type fixed, parent base_link, child depth_camera_link, origin xyz=0.2 0 0.1 rpy=0 0 0
